Commit message: modify topic name and frame_id for SLAM

File: velodyne_description/urdf/example.urdf.xacro (robot description, xacro)
@@ -1,38 +1,36 @@
 <?xml version="1.0"?>
 <robot xmlns:xacro="http://www.ros.org/wiki/xacro" name="example">
-  <!-- Base Footprint -->
-  <link name="base_footprint" />
   <!-- Base Link -->
   <joint name="footprint" type="fixed" >
-   <parent link="base_footprint" />
-    <child link="base_link" />
-    <origin xyz="0 0 0.05" rpy="0 0 0" />
+   <parent link="base_link" />
+    <child link="velo_base_link" />
+    <origin xyz="0.0 0 0.2" rpy="0 0 0" />
   </joint>
-  <link name="base_link" >
+  <link name="velo_base_link" >
     <visual>
       <geometry>
-        <box size="0.5 0.5 0.1" />
+        <box size="0.1 0.1 0.2" />
       </geometry>
     </visual>
     <collision>
       <geometry>
-        <box size="0.5 0.5 0.1" />
+        <box size="0.1 0.1 0.2" />
       </geometry>
     </collision>
     <inertial>
       <origin xyz="0 0 0"/>
-      <mass value="10"/>
-      <inertia ixx="3.0" ixy="0.0" ixz="0.0"
-               iyy="3.0" iyz="0.0"
-               izz="3.0" />
+      <mass value="0.001"/>
+      <inertia ixx="0.001" ixy="0.0" ixz="0.0"
+               iyy="0.001" iyz="0.0"
+               izz="0.001" />
     </inertial>
   </link>
   <xacro:include filename="$(find velodyne_description)/urdf/VLP-16.urdf.xacro"/>
-  <VLP-16 parent="base_link" name="velodyne" topic="/velodyne_points" hz="10" samples="440">
-    <origin xyz="0 0 0.4" rpy="0 0 0" />
+  <VLP-16 parent="velo_base_link" name="velodyne" topic="/velodyne_points" hz="10" samples="440">
+    <origin xyz="0 0 0.1" rpy="0 0 0" />
   </VLP-16>
-  <xacro:include filename="$(find velodyne_description)/urdf/HDL-32E.urdf.xacro"/>
+  <!--xacro:include filename="$(find velodyne_description)/urdf/HDL-32E.urdf.xacro"/>
   <HDL-32E parent="base_link" name="velodyne2" topic="/velodyne_points2" hz="10" samples="220">
     <origin xyz="0 0 0.6" rpy="0 0 0" />
-  </HDL-32E>
+  </HDL-32E-->
 </robot>
